Commit message: Copy FR3 and FT sensor support from melodic branch

File: config/arm.xacro (robot description, xacro)
@@ -67,3 +67,13 @@
     <xacro:configure_collisions link="6" />
     <xacro:configure_collisions link="7" />
+    <!-- Disable collision of FT sensor with all arm links  -->
+    <xacro:property name="link_fmt" value="$(arg arm_id)_link{}" />
+    <xacro:if value="$(arg use_FT_sensor)">
+        <xacro:disable_collisions_for link="$(arg FT_prefix)_mounting" others="${[link_fmt.format(i) for i in python.range(8)]}" />
+    </xacro:if>
+    <!-- Disable collision of FT sensor with all _sc links -->
+    <xacro:property name="link_fmt" value="$(arg arm_id)_link{}_sc" />
+    <xacro:if value="$(arg use_FT_sensor)">
+        <xacro:disable_collisions_for link="$(arg FT_prefix)_mounting" others="${[link_fmt.format(i) for i in python.range(8)]}" />
+    </xacro:if>
 </robot>

File: config/hand.xacro (robot description, xacro)
@@ -38,4 +38,11 @@
         <xacro:disable_collisions_for link="$(arg arm_id)_rightfinger" others="${list(others)}" />
         <disable_collisions link1="$(arg arm_id)_leftfinger" link2="$(arg arm_id)_rightfinger" reason="Never" />
+        <!-- Disable collision of FT sensor with hand and fingers -->
+        <xacro:if value="$(arg use_FT_sensor)">
+            <disable_collisions link1="$(arg FT_prefix)_mounting" link2="$(arg arm_id)_hand" reason="Never" />
+            <disable_collisions link1="$(arg FT_prefix)_mounting" link2="$(arg arm_id)_hand_sc" reason="Never" />
+            <disable_collisions link1="$(arg FT_prefix)_mounting" link2="$(arg arm_id)_rightfinger" reason="Never" />
+            <disable_collisions link1="$(arg FT_prefix)_mounting" link2="$(arg arm_id)_leftfinger" reason="Never" />
+        </xacro:if>
     </xacro:macro>
 </robot>

Commit message: Modify to support FR3 and FT sensor

File: config/arm.xacro (robot description, xacro)
@@ -59,3 +59,13 @@
     <xacro:configure_collisions link="6" />
     <xacro:configure_collisions link="7" />
+    <!-- Disable collision of FT sensor with all arm links  -->
+    <xacro:property name="link_fmt" value="$(arg arm_id)_link{}" />
+    <xacro:if value="$(arg use_FT_sensor)">
+        <xacro:disable_collisions_for link="$(arg FT_prefix)_mounting" others="${[link_fmt.format(i) for i in python.range(8)]}" />
+    </xacro:if>
+    <!-- Disable collision of FT sensor with all _sc links -->
+    <xacro:property name="link_fmt" value="$(arg arm_id)_link{}_sc" />
+    <xacro:if value="$(arg use_FT_sensor)">
+        <xacro:disable_collisions_for link="$(arg FT_prefix)_mounting" others="${[link_fmt.format(i) for i in python.range(8)]}" />
+    </xacro:if>
 </robot>

File: config/hand.xacro (robot description, xacro)
@@ -42,4 +42,11 @@
         <!-- Disable collision of hand_sc with selected arm sc links -->
         <xacro:disable_collisions_for link="$(arg arm_id)_hand_sc" others="${[link_fmt.format(i) for i in [4,5,6,7]]}" />
+        <!-- Disable collision of FT sensor with hand and fingers -->
+        <xacro:if value="$(arg use_FT_sensor)">
+            <disable_collisions link1="$(arg FT_prefix)_mounting" link2="$(arg arm_id)_hand" reason="Never" />
+            <disable_collisions link1="$(arg FT_prefix)_mounting" link2="$(arg arm_id)_hand_sc" reason="Never" />
+            <disable_collisions link1="$(arg FT_prefix)_mounting" link2="$(arg arm_id)_rightfinger" reason="Never" />
+            <disable_collisions link1="$(arg FT_prefix)_mounting" link2="$(arg arm_id)_leftfinger" reason="Never" />
+        </xacro:if>
     </xacro:macro>
 </robot>
